File: atx48.kicad_sch (KiCad schematic)
At the start: 84 parts, among them J1 XT60, J2 ATX-24, J3 Conn_02x02_Top_Bottom, J4 Conn_02x02_Top_Bottom, Q2 KIA3510AD, Q5 2N7002, Q6 2N7002, U1 Brick-DCDC, U10 ZXDN10, U2 LM5067, U3 EL3H7(B)(TA)-G, U4 EL3H7(B)(TA)-G, U5 AV10-48S05, U6 EL3H7(B)(TA)-G, U7 TPS3510, U8 ZXDN10, U9 ZXDN10

Commit message: Add filter capacitors; add Y cap
Parts:
- added C18, C19, C21, C22, C28: 10nF/100V, lc:0603_C, symbol Device:C_Small
- added C20, C27: 100nF/100V, lc:0805_C, symbol Device:C_Small
- added C23, C24, C29, C31, C33, C35, C36, C37, C38, C39, C40, C41, C43, C44, C46: 10nF, lc:0603_C, symbol Device:C_Small
- added C25, C26, C30, C32, C34, C45: 100nF, lc:0805_C, symbol Device:C_Small
- added C42: 1nF Y1, Capacitor_THT:C_Disc_D8.0mm_W5.0mm_P10.00mm, symbol Device:C_Small
- added F1: T10A, Fuse:Fuse_1812_4532Metric, symbol Device:Fuse
- FL1: value ACM1513F-551T100 -> ACM1513F-301T130
Connections:
- net +12V: now also C23.1, C24.1, C25.1, C26.1, C35.1, C36.1, C37.1, C38.1, C39.1, C40.1, C41.1, C43.1, C44.1, C45.1, C46.1
- net +3.3V: now also C33.1, C34.1
- net +5VA: now also C31.1, C32.1
- net +5VD: now also C29.1, C30.1
- net GND1: now also C19.2, C20.2, C21.2
- net GND2: now also C23.2, C24.2, C25.2, C26.2, C29.2, C30.2, C31.2, C32.2, C33.2, C34.2, C35.2, C36.2, C37.2, C38.2, C39.2, C40.2, C41.2, C42.2, C43.2, C44.2, C45.2, C46.2
- net NEG_FIL: now also C18.2, C22.2, C27.2, C28.2
- net RTN: now also C19.1, C20.1, C21.1, C42.1
- net RTN_FIL: now also C18.1, C22.1, C27.1, C28.1
- net VEE: now also F1.2; no longer J1.1 (Pin_1)
- new net: F1.1, J1.1 (Pin_1)
Other:
- moved on the sheet: C1, C10, C11, C12, C13, C14, C15, C16, C17, C2, C3, C4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
